File: hardware/buggyboy/brains.kicad_pcb (KiCad board)
At the start: 2 copper layers, 88 x 132 mm, 97 parts, among them J1 SCREEN_CONNECTOR, J2 Conn_01x04, J4 OUT, J5 MIC, J6 DEBUG_TELCO, SW1 SW_SPDT, U1 MT8888CN1, U2 LM386, U3 LM386, U4 LM66100, X1 CXO_DIP14

Commit message: routed again
Parts:
- removed D13, D14: WS2812B, LED_SMD:LED_WS2812B_PLCC4_5.0x5.0mm_P3.2mm
- removed the D2 at (145.5, 34.0)
- removed the D6 at (119.0, 157.0)
- removed the D7 at (109.0, 143.0)
- removed G***: LOGO, buggyboy:uwu
- removed G***: LOGO, buggyboy:smug_futaba
- removed G***: LOGO, buggyboy:smug_sans
- removed G***: LOGO, buggyboy:text
- removed JP1: JUMP_IDEAL_DIODE, Jumper:SolderJumper-2_P1.3mm_Open_RoundedPad1.0x1.5mm
- removed R10: 180R, Resistor_SMD:R_0805_2012Metric_Pad1.15x1.40mm_HandSolder
- removed R11: 290R, Resistor_SMD:R_0805_2012Metric_Pad1.15x1.40mm_HandSolder
- removed R12: 100k, Resistor_SMD:R_0805_2012Metric_Pad1.15x1.40mm_HandSolder
- removed REF**: SIG, buggyboy:SIG
- removed RV_MIC1, RV_VOLUME1: 10k, Potentiometer_THT:Potentiometer_Bourns_PTV09A-2_Single_Horizontal
- removed TP5: TP_DIODE_BATT, TestPoint:TestPoint_Pad_D2.5mm
- removed U4: LM66100, Package_TO_SOT_SMD:SOT-363_SC-70-6_Handsoldering
- added D10: WS2812B, LED_SMD:LED_WS2812B_PLCC4_5.0x5.0mm_P3.2mm, F.Cu at (186.0, 75.0)
- added D41: DZener, Diode_SMD:D_SMB_Handsoldering, F.Cu at (160.0, 146.0)
- added D42: D, Diode_SMD:D_SMA_Handsoldering, F.Cu at (160.0, 141.0)
- added D5: WS2812B, LED_SMD:LED_WS2812B_PLCC4_5.0x5.0mm_P3.2mm, F.Cu at (110.0, 127.0)
- added D9: WS2812B, LED_SMD:LED_WS2812B_PLCC4_5.0x5.0mm_P3.2mm, F.Cu at (186.0, 49.0)
- added F2: Polyfuse, Fuse:Fuse_Littelfuse_395Series, F.Cu at (172.5, 146.0)
- added H3: MNT3, MountingHole:MountingHole_4.3mm_M4_Pad_Via, F.Cu at (187.0, 35.0)
- added H4: MNT4, MountingHole:MountingHole_4.3mm_M4_Pad_Via, F.Cu at (109.0, 35.0)
- added JP3: JUMP_ZENER, Jumper:SolderJumper-2_P1.3mm_Open_RoundedPad1.0x1.5mm, F.Cu at (159.8, 149.5)
- added JP4: JUMP_PF, Jumper:SolderJumper-2_P1.3mm_Open_RoundedPad1.0x1.5mm, F.Cu at (170.0, 150.5)
- added JP5: BP_C, Jumper:SolderJumper-2_P1.3mm_Open_RoundedPad1.0x1.5mm, F.Cu at (172.9, 74.9)
- added JP6: BP_R, Jumper:SolderJumper-2_P1.3mm_Open_RoundedPad1.0x1.5mm, F.Cu at (176.9, 74.9)
- added JP7: JUMP_MIC_OUT_CAP, Jumper:SolderJumper-2_P1.3mm_Open_RoundedPad1.0x1.5mm, F.Cu at (166.8, 79.5)
- BT1: footprint Battery:BatteryHolder_BC2AAPC -> buggyboy:BatteryHolder_BC2AAPC; moved to B.Cu
- C1: value 100nF -> 10uF; footprint Capacitor_SMD:C_0805_2012Metric_Pad1.15x1.40mm_HandSolder -> Capacitor_SMD:C_0805_2012Metric_Pad1.18x1.45mm_HandSolder
- C10: value 100nF -> 47nF; footprint Capacitor_SMD:C_0805_2012Metric_Pad1.15x1.40mm_HandSolder -> Capacitor_SMD:C_0805_2012Metric
- C11, C17, C21: footprint Capacitor_SMD:C_1210_3225Metric_Pad1.33x2.70mm_HandSolder -> Capacitor_SMD:C_1206_3216Metric_Pad1.33x1.80mm_HandSolder
- C12, C18, C23, C24, C25, C26, C27, C28, C29, C3, C30, C31, C32, C4, C6, C9: footprint Capacitor_SMD:C_0805_2012Metric_Pad1.15x1.40mm_HandSolder -> Capacitor_SMD:C_0603_1608Metric_Pad1.08x0.95mm_HandSolder
- C13, C14, C15, C2, C20: footprint Capacitor_SMD:C_0805_2012Metric_Pad1.15x1.40mm_HandSolder -> Capacitor_SMD:C_0805_2012Metric_Pad1.18x1.45mm_HandSolder
- C16: value 10uF -> DEPOP; footprint Capacitor_SMD:C_0805_2012Metric_Pad1.15x1.40mm_HandSolder -> Capacitor_THT:CP_Radial_D8.0mm_P3.80mm
- C19: value 10uF -> 100nF; footprint Capacitor_SMD:C_0805_2012Metric_Pad1.15x1.40mm_HandSolder -> Capacitor_SMD:C_0603_1608Metric_Pad1.08x0.95mm_HandSolder
- C22: value 100uF -> 100nF; footprint Capacitor_SMD:C_1210_3225Metric_Pad1.33x2.70mm_HandSolder -> Capacitor_SMD:C_0603_1608Metric_Pad1.08x0.95mm_HandSolder
- C5: value 100nF -> DEPOP; footprint Capacitor_SMD:C_0805_2012Metric_Pad1.15x1.40mm_HandSolder -> Capacitor_THT:CP_Radial_D8.0mm_P3.80mm
- C7: value 100nF -> 10uF; footprint Capacitor_SMD:C_0805_2012Metric_Pad1.15x1.40mm_HandSolder -> Capacitor_SMD:C_0805_2012Metric
- C8: value 100nF -> 470uF; footprint Capacitor_SMD:C_0805_2012Metric_Pad1.15x1.40mm_HandSolder -> Capacitor_THT:CP_Radial_D8.0mm_P3.80mm
- D1: value GREEN -> WS2812B; footprint LED_THT:LED_D5.0mm_Horizontal_O3.81mm_Z3.0mm -> LED_SMD:LED_WS2812B_PLCC4_5.0x5.0mm_P3.2mm
- J4, J5: footprint Connector_Audio:CUI_SJ1-3545N -> buggyboy:CUI_SJ1-3545N
- R1, R14, R15, R4, R5, R6, R8, R9: footprint Resistor_SMD:R_0805_2012Metric_Pad1.15x1.40mm_HandSolder -> Resistor_SMD:R_0805_2012Metric_Pad1.20x1.40mm_HandSolder
- R2: value 100k -> 9.7k; footprint Resistor_SMD:R_0805_2012Metric_Pad1.15x1.40mm_HandSolder -> Resistor_SMD:R_0805_2012Metric_Pad1.20x1.40mm_HandSolder
- R3: value 470 -> 1k; footprint Resistor_SMD:R_0805_2012Metric_Pad1.15x1.40mm_HandSolder -> Resistor_SMD:R_0805_2012Metric_Pad1.20x1.40mm_HandSolder
- R7: value 1k -> 10k; footprint Resistor_SMD:R_0805_2012Metric_Pad1.15x1.40mm_HandSolder -> Resistor_SMD:R_0805_2012Metric_Pad1.20x1.40mm_HandSolder
- U1: footprint Package_SO:SSOP-24_5.3x8.2mm_P0.65mm -> buggyboy:SSOP-24_5.3x8.2mm_P0.65mm-HandSolder
- moved D1 125.3 mm to (177.0, 157.0), turned to 0 degrees
- moved D4 112.4 mm to (119.0, 157.0)
- moved D11 84.6 mm to (186.0, 101.0)
- moved C26 84.3 mm to (184.1, 97.0), turned to 180 degrees
- moved C7 80.4 mm to (177.6, 62.2), turned to 180 degrees
- moved C23 78.0 mm to (184.0, 140.0), turned to 180 degrees
- moved D12 78.0 mm to (186.0, 144.0)
- moved C24 77.5 mm to (108.1, 45.0), turned to 180 degrees
- moved D8 77.1 mm to (110.0, 49.0)
- moved D6 60.2 mm to (110.0, 101.0)
- moved C25 56.0 mm to (108.1, 97.0), turned to 180 degrees
- moved JP2 52.5 mm to (131.5, 53.0)
- moved C19 49.0 mm to (184.0, 45.0), turned to 180 degrees
- moved R2 47.1 mm to (116.7, 114.3)
- moved D3 45.0 mm to (132.0, 157.0)
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- renumbered D9 to D11, D4 to D2, D10 to D4, D5 to D6, D8 to D7, D11 to D8
Connections:
- A1 pad 1: Net-(A1-Pad1) -> (no net)
- A1 pad 17: Net-(A1-Pad17) -> (no net)
- A1 pad 18: Net-(A1-Pad18) -> (no net)
- A1 pad 2: Net-(A1-Pad2) -> (no net)
- A1 pad 23: Net-(A1-Pad23) -> (no net)
- A1 pad 24: Net-(A1-Pad24) -> (no net)
- A1 pad 25: Net-(A1-Pad25) -> (no net)
- A1 pad 26: Net-(A1-Pad26) -> (no net)
- A1 pad 28: Net-(A1-Pad28) -> (no net)
- A1 pad 3: Net-(A1-Pad3) -> (no net)
- A1 pad 8: Net-(A1-Pad8) -> (no net)
- A1 pad 9: /NEOPIXELS -> /NEOPIXEL
- C16 pad 2: Net-(C16-Pad2) -> GND
- C19 pad 1: Net-(C19-Pad1) -> GND
- C19 pad 2: GND -> +5V
- C22 pad 1: Net-(C22-Pad1) -> GND
- C22 pad 2: Net-(C10-Pad1) -> +5V
- C23 pad 1: +5V -> GND
- C23 pad 2: GND -> +5V
- C24 pad 1: +5V -> GND
- C24 pad 2: GND -> +5V
- C25 pad 1: +5V -> GND
- C25 pad 2: GND -> +5V
- C26 pad 1: +5V -> GND
- C26 pad 2: GND -> +5V
- C27 pad 1: +5V -> GND
- C27 pad 2: GND -> +5V
- C28 pad 1: +5V -> GND
- C28 pad 2: GND -> +5V
- C29 pad 1: +5V -> GND
- C29 pad 2: GND -> +5V
- C30 pad 1: +5V -> GND
- C30 pad 2: GND -> +5V
- C31 pad 1: +5V -> GND
- C31 pad 2: GND -> +5V
- C32 pad 1: +5V -> GND
- C32 pad 2: GND -> +5V
- C7 pad 1: +5V -> GND
- C7 pad 2: GND -> Net-(C16-Pad1)
- C8 pad 1: +5V -> Net-(C10-Pad1)
- C8 pad 2: GND -> Net-(C8-Pad2)
- D1 pad 1: GND -> +5V
- D11 pad 2: Net-(D10-Pad4) -> Net-(D11-Pad2)
- D11 pad 4: Net-(D8-Pad2) -> Net-(D10-Pad2)
- D2 pad 2: Net-(D4-Pad2) -> Net-(D2-Pad2)
- D2 pad 4: Net-(D3-Pad2) -> Net-(D1-Pad2)
- D3 pad 4: Net-(D3-Pad4) -> Net-(D2-Pad2)
- D4 pad 2: Net-(D10-Pad2) -> Net-(D4-Pad2)
- D4 pad 4: Net-(D10-Pad4) -> Net-(D3-Pad2)
- D6 pad 2: Net-(D5-Pad2) -> Net-(D6-Pad2)
- D6 pad 4: Net-(D4-Pad2) -> Net-(D5-Pad2)
- D7 pad 2: Net-(D8-Pad2) -> Net-(D7-Pad2)
- D7 pad 4: Net-(D7-Pad2) -> Net-(D6-Pad2)
- D8 pad 2: Net-(D11-Pad2) -> Net-(D8-Pad2)
- D8 pad 4: Net-(D10-Pad2) -> Net-(D7-Pad2)
- F1 pad 1: Net-(BT1-Pad1) -> Net-(D42-Pad2)
- F1 pad 2: Net-(F1-Pad2) -> GND
- J4 pad 5: Net-(J4-Pad4) -> (no net)
- J5 pad 2: Net-(C22-Pad1) -> Net-(C8-Pad2)
- J5 pad 3: Net-(C22-Pad1) -> Net-(C8-Pad2)
- J5 pad 4: Net-(C1-Pad2) -> /DTMF_IN
- J5 pad 5: Net-(C1-Pad2) -> (no net)
- MK1 pad 2: Net-(C5-Pad2) -> Net-(C1-Pad2)
- R2 pad 1: Net-(R2-Pad1) -> /DTMF_OUT
- R2 pad 2: Net-(C1-Pad1) -> Net-(R2-Pad2)
- R3 pad 1: /NEOPIXELS -> GND
- R3 pad 2: Net-(D3-Pad4) -> Net-(D12-Pad2)
- R4 pad 2: Net-(R2-Pad1) -> /DTMF_IN
- R7 pad 1: +5V -> Net-(C1-Pad2)
- R7 pad 2: Net-(C5-Pad2) -> +5V
- SW1 pad 1: Net-(SW1-Pad1) -> (no net)
- SW1 pad 2: Net-(F1-Pad2) -> Net-(BT1-Pad1)
- TP1 pad 1: Net-(R2-Pad1) -> /DTMF_IN
- U1 pad 16: Net-(U1-Pad16) -> (no net)
- U1 pad 17: Net-(U1-Pad17) -> (no net)
- U1 pad 2: Net-(R2-Pad1) -> /DTMF_IN
- U1 pad 7: Net-(U1-Pad7) -> (no net)
- U1 pad 8: Net-(U1-Pad8) -> (no net)
- U1 pad 9: Net-(U1-Pad9) -> (no net)
- U2 pad 3: Net-(RV_VOLUME1-Pad2) -> Net-(R2-Pad2)
- U3 pad 1: Net-(C16-Pad1) -> Net-(C5-Pad1)
- U3 pad 3: Net-(RV_MIC1-Pad2) -> Net-(C1-Pad1)
- U3 pad 7: Net-(C19-Pad1) -> Net-(C16-Pad1)
- U3 pad 8: Net-(C16-Pad2) -> Net-(C5-Pad2)
Routing:
- net +5V: track 620.6 -> 472.2 mm, vias 5 -> 1
- net Net-(C5-Pad1): track 151.0 -> 9.98 mm, vias 4 -> 0
- net Net-(A1-Pad24): track 90.1 -> 0.00 mm, vias 3 -> 0
- net Net-(RV_MIC1-Pad2): track 88.7 -> 0.00 mm, vias 2 -> 0
- net Net-(C22-Pad1): track 88.5 -> 0.00 mm, vias 1 -> 0
- net Net-(A1-Pad23): track 85.8 -> 0.00 mm, vias 3 -> 0
- net Net-(D10-Pad2): track 109.2 -> 24.8 mm
- net Net-(D8-Pad2): track 26.4 -> 94.0 mm, vias 0 -> 2
- net /DTMF_IN: track 0.00 -> 65.5 mm
- net Net-(D13-Pad2): track 56.2 -> 0.00 mm
- net GND: track 46.2 -> 13.9 mm, vias 155 -> 24
- net Net-(D7-Pad2): track 63.1 -> 31.2 mm
- net Net-(C1-Pad2): track 65.4 -> 34.1 mm, vias 2 -> 0
- net Net-(R2-Pad1): track 28.1 -> 0.00 mm
- net /NEOPIXEL: track 0.00 -> 26.9 mm, vias 0 -> 2
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Other:
- outline, holes or cut-outs redrawn
- board text removed: ">2022 >gonna be my year"
- board text removed: "GREEN"
- board text removed: "MIC"
- board text removed: "RED"
- board text removed: "VOL"
- board text removed: "be gay do crimes"
- board text removed: "hewwo!"

Commit message: ordering
Parts:
- added C33: 32pF, Capacitor_SMD:C_0402_1005Metric_Pad0.74x0.62mm_HandSolder, F.Cu at (167.2, 98.9)
- added C34: 32pF, Capacitor_SMD:C_0402_1005Metric_Pad0.74x0.62mm_HandSolder, F.Cu at (173.1, 99.0)
- added C35: 100nF, Capacitor_SMD:C_0603_1608Metric_Pad1.08x0.95mm_HandSolder, F.Cu at (175.2, 94.9)
- added JP1: JUMP_XTAL_ALT, Jumper:SolderJumper-2_P1.3mm_Open_RoundedPad1.0x1.5mm, F.Cu at (175.1, 92.4)
- added R10: 2.2m, Resistor_SMD:R_0805_2012Metric_Pad1.20x1.40mm_HandSolder, F.Cu at (170.1, 98.4)
- added U4: SN74LVC1GX04, Package_TO_SOT_SMD:SOT-563, F.Cu at (170.1, 95.4)
- added Y1: Crystal_Small, Crystal:Crystal_HC49-U_Vertical, F.Cu at (163.4, 89.8)
- C10: footprint Capacitor_SMD:C_0805_2012Metric -> Capacitor_SMD:C_0603_1608Metric_Pad1.08x0.95mm_HandSolder
- C7: footprint Capacitor_SMD:C_0805_2012Metric -> Capacitor_SMD:C_0805_2012Metric_Pad1.18x1.45mm_HandSolder
- U1: value MT8888CN1 -> MT8888CS1; footprint buggyboy:SSOP-24_5.3x8.2mm_P0.65mm-HandSolder -> Package_SO:SOIC-20W_7.5x12.8mm_P1.27mm
- moved C3 10.1 mm to (130.5, 89.7), turned to 180 degrees
- moved C4 7.42 mm to (130.8, 87.7), turned to 0 degrees
- moved R6 5.24 mm to (130.8, 85.7), turned to 0 degrees
- moved U1 5.22 mm to (140.3, 83.7)
- moved R5 0.85 mm to (146.8, 74.8)
- moved J5 0.20 mm to (167.4, 33.3)
Connections:
- A1 pad 1: (no net) -> Net-(A1-Pad1)
- A1 pad 17: (no net) -> Net-(A1-Pad17)
- A1 pad 18: (no net) -> Net-(A1-Pad18)
- A1 pad 2: (no net) -> Net-(A1-Pad2)
- A1 pad 23: (no net) -> Net-(A1-Pad23)
- A1 pad 24: (no net) -> Net-(A1-Pad24)
- A1 pad 25: (no net) -> Net-(A1-Pad25)
- A1 pad 26: (no net) -> Net-(A1-Pad26)
- A1 pad 28: (no net) -> Net-(A1-Pad28)
- A1 pad 3: (no net) -> Net-(A1-Pad3)
- A1 pad 8: (no net) -> Net-(A1-Pad8)
- J4 pad 5: (no net) -> Net-(J4-Pad4)
- J5 pad 5: (no net) -> /DTMF_IN
- SW1 pad 1: (no net) -> Net-(SW1-Pad1)
- U1 pad 10: Net-(C2-Pad2) -> /TELCO_CS
- U1 pad 11: /TELCO_WR -> /TELCO_RS0
- U1 pad 12: /TELCO_CS -> /TELCO_RD
- U1 pad 13: /TELCO_RS0 -> /TELCO_IRQ
- U1 pad 14: /TELCO_RD -> /D0
- U1 pad 15: /TELCO_IRQ -> /D1
- U1 pad 16: (no net) -> /D2
- U1 pad 17: (no net) -> /D3
- U1 pad 18: /D0 -> Net-(R6-Pad1)
- U1 pad 19: /D1 -> Net-(C4-Pad2)
- U1 pad 20: /D2 -> +5V
- U1 pad 7: (no net) -> Net-(U1-Pad7)
- U1 pad 8: (no net) -> Net-(C2-Pad2)
- U1 pad 9: (no net) -> /TELCO_WR
Routing:
- net +5V: track 472.2 -> 578.3 mm, vias 1 -> 3
- net Net-(C8-Pad2): track 20.8 -> 64.7 mm, vias 0 -> 1
- net Net-(JP1-Pad2): track 30.4 -> 60.9 mm
- net GND: track 13.9 -> 37.4 mm, vias 24 -> 41
- net Net-(C33-Pad2): track 0.00 -> 14.7 mm
- net Net-(C34-Pad2): track 0.00 -> 13.2 mm
- net /DISP_RS: track 103.5 -> 115.5 mm
- net /DISP_EN: track 104.6 -> 116.5 mm
- net /DTMF_IN: track 65.5 -> 75.9 mm
- net Net-(J4-Pad4): track 13.4 -> 19.6 mm
- net /D3: track 125.4 -> 130.3 mm
- net /XTAL_ALT: track 0.00 -> 4.63 mm
- net /D0: track 110.2 -> 114.7 mm
- net /D2: track 118.2 -> 122.5 mm
- net /D1: track 112.3 -> 116.5 mm
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Other:
- board text removed: "+"
- board text removed: "-"
- board text removed: "3.579545MHz"
- board text removed: "What de fack did yuw just facking say about me, yuw wittwe bitch? I’ww have yuw know I gwaduated top of my cwass in de Navy Seaws, and I’ve been invowved in numewous secwet waids on Aw-Quaeda, and I have ovew 300 confiwmed kiwws. I am twained in gowiwwa wawfawe and I’m de top snipew in de entiwe US awmed fowces. yuw awe nofing to me but just anofew tawget. I wiww wipe yuw de fack out wif pwecisio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"
