File: hardware/buggyboy/brains.sch (KiCad schematic (older format))
At the start: 108 parts, among them J1 SCREEN_CONNECTOR, J2 Conn_01x04, J4 OUT, J5 MIC, J6 DEBUG_TELCO, Q1 IRL540, Q2 IRL540, SW1 SW_SPDT, U1 MT8888CN1, U2 LM386, U3 LM386, U4 LM66100, X1 CXO_DIP14

Commit message: before redoin
Parts:
- removed C16: 10uF, Capacitor_SMD:C_0805_2012Metric_Pad1.15x1.40mm_HandSolder, symbol Device:C_Small
- removed C5: 100nF, Capacitor_SMD:C_0805_2012Metric_Pad1.15x1.40mm_HandSolder, symbol Device:C_Small
- removed D1, D10, D11, D12, D13, D14, D15, D16, D17, D18, D19, D2, D20, D3, D4, D5, D6, D7, D8, D9: BLUE, LED_SMD:LED_0805_2012Metric_Pad1.15x1.40mm_HandSolder, symbol Device:LED
- removed D21, D22, D23, D24, D25, D26, D27, D28, D29, D30, D31, D32, D33, D34, D35, D36, D37, D38, D39, D40: RED, LED_SMD:LED_0603_1608Metric_Pad1.05x0.95mm_HandSolder, symbol Device:LED
- removed Q1, Q2: IRL540, symbol tinkerforge:MOSFET_N_CH
- removed R10: 100, symbol Device:R
- removed R11: 10k, Resistor_SMD:R_0805_2012Metric_Pad1.15x1.40mm_HandSolder, symbol Device:R
- removed R12: 150, symbol Device:R
- removed RV_MIC1, RV_VOLUME1: 10k, Potentiometer_THT:Potentiometer_Bourns_PTV09A-2_Single_Horizontal, symbol Device:R_POT
- added C16, C5: DEPOP, Capacitor_THT:CP_Radial_D8.0mm_P3.80mm, symbol Device:CP_Small
- added C23, C24, C25, C26, C27, C28, C29, C30, C31, C32: 100nF, Capacitor_SMD:C_0603_1608Metric_Pad1.08x0.95mm_HandSolder, symbol Device:C_Small
- added C7: 10uF, Capacitor_SMD:C_0805_2012Metric, symbol Device:C_Small
- added C8: 470uF, Capacitor_THT:CP_Radial_D8.0mm_P3.80mm, symbol Device:CP_Small
- added D1, D10, D11, D12, D2, D3, D4, D5, D6, D7, D8, D9: WS2812B, LED_SMD:LED_WS2812B_PLCC4_5.0x5.0mm_P3.2mm, symbol LED:WS2812B
- added D41: D_Zener_Small, Diode_SMD:D_SMB_Handsoldering, symbol Device:D_Zener_Small
- added D42: D, Diode_SMD:D_SMA_Handsoldering, symbol Device:D
- added F2: Polyfuse, Fuse:Fuse_Littelfuse_395Series, symbol Device:Polyfuse
- added H3: MNT3, MountingHole:MountingHole_4.3mm_M4_Pad_Via, symbol Mechanical:MountingHole_Pad
- added H4: MNT4, MountingHole:MountingHole_4.3mm_M4_Pad_Via, symbol Mechanical:MountingHole_Pad
- added JP3: JUMP_ZENER, Jumper:SolderJumper-2_P1.3mm_Open_RoundedPad1.0x1.5mm, symbol Jumper:Jumper_2_Open
- added JP4: JUMP_PF, Jumper:SolderJumper-2_P1.3mm_Open_RoundedPad1.0x1.5mm, symbol Jumper:Jumper_2_Open
- added JP5: BP_C, Jumper:SolderJumper-2_P1.3mm_Open_RoundedPad1.0x1.5mm, symbol Device:Jumper_NO_Small
- added JP6: BP_R, Jumper:SolderJumper-2_P1.3mm_Open_RoundedPad1.0x1.5mm, symbol Device:Jumper_NO_Small
- added JP7: JUMP_MIC_OUT_CAP, Jumper:SolderJumper-2_P1.3mm_Open_RoundedPad1.0x1.5mm, symbol Device:Jumper_NO_Small
- BT1: footprint Battery:BatteryHolder_BC2AAPC -> buggyboy:BatteryHolder_BC2AAPC
- C1: value 100nF -> 10uF; footprint Capacitor_SMD:C_0805_2012Metric_Pad1.15x1.40mm_HandSolder -> Capacitor_SMD:C_0805_2012Metric_Pad1.18x1.45mm_HandSolder
- C10: value 100nF -> 47nF; footprint Capacitor_SMD:C_0805_2012Metric_Pad1.15x1.40mm_HandSolder -> Capacitor_SMD:C_0805_2012Metric
- C11, C17, C21: footprint Capacitor_SMD:C_1210_3225Metric_Pad1.33x2.70mm_HandSolder -> Capacitor_SMD:C_1206_3216Metric_Pad1.33x1.80mm_HandSolder
- C12, C18, C3, C4, C6, C9: footprint Capacitor_SMD:C_0805_2012Metric_Pad1.15x1.40mm_HandSolder -> Capacitor_SMD:C_0603_1608Metric_Pad1.08x0.95mm_HandSolder
- C13, C14, C15, C2, C20: footprint Capacitor_SMD:C_0805_2012Metric_Pad1.15x1.40mm_HandSolder -> Capacitor_SMD:C_0805_2012Metric_Pad1.18x1.45mm_HandSolder
- C19: value 10uF -> 100nF; footprint Capacitor_SMD:C_0805_2012Metric_Pad1.15x1.40mm_HandSolder -> Capacitor_SMD:C_0603_1608Metric_Pad1.08x0.95mm_HandSolder
- C22: value 100uF -> 100nF; footprint Capacitor_SMD:C_1210_3225Metric_Pad1.33x2.70mm_HandSolder -> Capacitor_SMD:C_0603_1608Metric_Pad1.08x0.95mm_HandSolder
- J4, J5: footprint Connector_Audio:CUI_SJ1-3545N -> buggyboy:CUI_SJ1-3545N
- R1, R14, R15, R4, R5, R6, R8, R9: footprint Resistor_SMD:R_0805_2012Metric_Pad1.15x1.40mm_HandSolder -> Resistor_SMD:R_0805_2012Metric_Pad1.20x1.40mm_HandSolder
- R2: value 100k -> 9.7k; footprint Resistor_SMD:R_0805_2012Metric_Pad1.15x1.40mm_HandSolder -> Resistor_SMD:R_0805_2012Metric_Pad1.20x1.40mm_HandSolder
- R3: value 10k -> 1k; footprint Resistor_SMD:R_0805_2012Metric_Pad1.15x1.40mm_HandSolder -> Resistor_SMD:R_0805_2012Metric_Pad1.20x1.40mm_HandSolder
- R7: value 1k -> 10k; footprint Resistor_SMD:R_0805_2012Metric_Pad1.15x1.40mm_HandSolder -> Resistor_SMD:R_0805_2012Metric_Pad1.20x1.40mm_HandSolder
- U1: symbol buggyboy:MT8888C -> brains-rescue:MT8888C-buggyboy
- U4: symbol buggyboy:LM66100 -> brains-rescue:LM66100-buggyboy
Connections:
- net labels added: NEOPIXEL
- net labels removed: BLUE, GREEN, RED
- wire segments 335 -> 298
Other:
- moved on the sheet: BT1, C10, C11, C12, C13, C14, C15, C17, C18, C20, C21, C6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

Commit message: routed again
Parts:
- removed JP1: JUMP_IDEAL_DIODE, Jumper:SolderJumper-2_P1.3mm_Open_RoundedPad1.0x1.5mm, symbol Jumper:Jumper_2_Open
- removed TP5: TP_DIODE_BATT, TestPoint:TestPoint_Pad_D2.5mm, symbol Connector:TestPoint
- removed U4: LM66100, Package_TO_SOT_SMD:SOT-363_SC-70-6_Handsoldering, symbol brains-rescue:LM66100-buggyboy
- D41: value D_Zener_Small -> DZener
- renumbered D6 to D10, D9 to D11, D4 to D2, D7 to D3, D10 to D4, D2 to D5, D5 to D6, D8 to D7, D11 to D8, D3 to D9
Connections:
- net at SW1.3 (C), TP6.1: now also F2.1, JP4.2 (B)
- no-connect marks 5 -> 4
Other:
- moved on the sheet: BT1, SW1, TP6
Changed lines of the file:
@@
-$EndComp
-$Comp
-L Switch:SW_SPDT SW1
-U 1 1 60E5AE6E
-P 11400 1450
-AR Path="/60E5AE6E" Ref="SW1"  Part="1"
-AR Path="/60E4053B/60E5AE6E" Ref="SW1"  Part="1"
-F 0 "SW1" H 11400 1125 50  0000 C CNN
-F 1 "SW_SPDT" H 11400 1216 50  0000 C CNN
-F 2 "Button_Switch_THT:SW_E-Switch_EG1224_SPDT_Angled" H 11400 1450 50  0001 C CNN
-F 3 "" H 11400 1450 50  0001 C CNN
-	1    11400 1450
-	-1   0    0    1
 $EndComp
 $Comp
@@
 L power:GND #PWR0119
 U 1 1 60E6EECF
-P 10650 2000
-F 0 "#PWR0119" H 10650 1750 50  0001 C CNN
-F 1 "GND" H 10655 1827 50  0000 C CNN
-F 2 "" H 10650 2000 50  0001 C CNN
-F 3 "" H 10650 2000 50  0001 C CNN
-	1    10650 2000
+P 9250 2000
+F 0 "#PWR0119" H 9250 1750 50  0001 C CNN
+F 1 "GND" H 9255 1827 50  0000 C CNN
+F 2 "" H 9250 2000 50  0001 C CNN
+F 3 "" H 9250 2000 50  0001 C CNN
+	1    9250 2000
 	1    0    0    -1
 $EndComp
@@
 NoConn ~ 6700 2300
 NoConn ~ 6700 2400
-$Comp
-L brains-rescue:LM66100-buggyboy U4
-U 1 1 61813B73
-P 10600 2400
-F 0 "U4" H 10600 3715 50  0000 C CNN
-F 1 "LM66100" H 10600 3624 50  0000 C CNN
-F 2 "Package_TO_SOT_SMD:SOT-363_SC-70-6_Handsoldering" H 10600 3300 50  0001 C CNN
-F 3 "" H 10600 3300 50  0001 C CNN
-	1    10600 2400
-	-1   0    0    -1
-$EndComp
-Wire Wire Line
-	11100 1350 11150 1350
-Wire Wire Line
-	10650 1900 10650 1950
-Wire Wire Line
-	10100 1500 10100 1950
-Wire Wire Line
-	10100 1950 10650 1950
-Connection ~ 10650 1950
-Wire Wire Line
-	10650 1950 10650 2000
-Wire Wire Line
-	11100 1950 11100 1500
-Wire Wire Line
-	10650 1950 11100 1950
-Connection ~ 10100 1950
-NoConn ~ 10500 1900
+Wire Wire Line
+	9250 1950 9250 2000
 $Comp
 L power:GND #PWR0108
@@
 L Connector:TestPoint TP6
 U 1 1 61253A17
-P 11150 1050
-F 0 "TP6" H 11208 1170 50  0000 L CNN
-F 1 "TP_RAW_BATT" H 11208 1079 50  0000 L CNN
-F 2 "TestPoint:TestPoint_Pad_D2.5mm" H 11350 1050 50  0001 C CNN
-F 3 "~" H 11350 1050 50  0001 C CNN
-	1    11150 1050
-	1    0    0    -1
-$EndComp
-Wire Wire Line
-	11150 1050 11150 1350
-Connection ~ 11150 1350
-Wire Wire Line
-	11150 1350 11200 1350
-$Comp
-L Connector:TestPoint TP5
-U 1 1 6126EBC1
-P 10050 1050
-F 0 "TP5" H 10108 1170 50  0000 L CNN
-F 1 "TP_DIODE_BATT" H 10108 1079 50  0000 L CNN
-F 2 "TestPoint:TestPoint_Pad_D2.5mm" H 10250 1050 50  0001 C CNN
-F 3 "~" H 10250 1050 50  0001 C CNN
-	1    10050 1050
-	1    0    0    -1
-$EndComp
-Wire Wire Line
-	10050 1050 10050 1350
-Connection ~ 10050 1350
-Wire Wire Line
-	10050 1350 10100 1350
+P 10000 950
+F 0 "TP6" H 10058 1070 50  0000 L CNN
+F 1 "TP_RAW_BATT" H 10058 979 50  0000 L CNN
+F 2 "TestPoint:TestPoint_Pad_D2.5mm" H 10200 950 50  0001 C CNN
+F 3 "~" H 10200 950 50  0001 C CNN
+	1    10000 950
+	1    0    0    -1
+$EndComp
+Wire Wire Line
+	10000 950  10000 1250
 $Comp
 L Connector:TestPoint TP4
@@
 	5150 1150 5150 950
 $Comp
-L Jumper:Jumper_2_Open JP1
-U 1 1 613557B2
-P 10600 850
-F 0 "JP1" H 10600 1085 50  0000 C CNN
-F 1 "JUMP_IDEAL_DIODE" H 10600 994 50  0000 C CNN
-F 2 "Jumper:SolderJumper-2_P1.3mm_Open_RoundedPad1.0x1.5mm" H 10600 850 50  0001 C CNN
-F 3 "~" H 10600 850 50  0001 C CNN
-	1    10600 850
-	1    0    0    -1
-$EndComp
-Wire Wire Line
-	10800 850  11200 850
-Wire Wire Line
-	11200 850  11200 1350
-Wire Wire Line
-	10400 850  10000 850
-Wire Wire Line
-	10000 850  10000 1250
-Wire Wire Line
-	10000 1350 10050 1350
-$Comp
 L Oscillator:CXO_DIP14 X1
 U 1 1 61D14DFF
@@
 L Device:Battery_Cell BT1
 U 1 1 621D61B0
-P 11900 1650
-F 0 "BT1" H 12018 1746 50  0000 L CNN
-F 1 "Battery_Cell" H 12018 1655 50  0000 L CNN
-F 2 "buggyboy:BatteryHolder_BC2AAPC" V 11900 1710 50  0001 C CNN
-F 3 "~" V 11900 1710 50  0001 C CNN
-	1    11900 1650
-	1    0    0    -1
-$EndComp
-Wire Wire Line
-	11900 1750 11900 1950
+P 10850 1550
+F 0 "BT1" H 10968 1646 50  0000 L CNN
+F 1 "Battery_Cell" H 10968 1555 50  0000 L CNN
+F 2 "buggyboy:BatteryHolder_BC2AAPC" V 10850 1610 50  0001 C CNN
+F 3 "~" V 10850 1610 50  0001 C CNN
+	1    10850 1550
+	1    0    0    -1
+$EndComp
 $Comp
 L brains-rescue:AudioJack2_Ground_Switch-buggyboy J5
@@
 	4750 1150 5150 1150
 Wire Wire Line
-	11600 1450 11900 1450
-Connection ~ 11200 1350
+	10550 1350 10850 1350
 $Comp
 L Device:D D42
 U 1 1 62D87177
 P 9250 1400
-F 0 "D42" V 9204 1480 50  0000 L CNN
-F 1 "D" V 9295 1480 50  0000 L CNN
+F 0 "D42" V 9200 1500 50  0000 L CNN
+F 1 "D" V 9300 1500 50  0000 L CNN
 F 2 "Diode_SMD:D_SMA_Handsoldering" H 9250 1400 50  0001 C CNN
 F 3 "~" H 9250 1400 50  0001 C CNN
@@
 Wire Wire Line
 	9250 1900 9250 1950
-Connection ~ 10000 1250
-Wire Wire Line
-	10000 1250 10000 1350
 $Comp
 L Device:D_Zener_Small D41
 U 1 1 62E71EDB
 P 9000 1250
-F 0 "D41" H 9000 1457 50  0000 C CNN
-F 1 "D_Zener_Small" H 9000 1366 50  0000 C CNN
+F 0 "D41" H 9000 1500 50  0000 C CNN
+F 1 "DZener" H 9000 1400 50  0000 C CNN
 F 2 "Diode_SMD:D_SMB_Handsoldering" V 9000 1250 50  0001 C CNN
 F 3 "~" V 9000 1250 50  0001 C CNN
@@
 	8800 900  8800 1250
 Connection ~ 8800 1250
-Wire Wire Line
-	11100 1950 11900 1950
-Connection ~ 11100 1950
 $Comp
 L Device:Polyfuse F2
@@
 Wire Wire Line
 	9650 1250 9700 1250
-Wire Wire Line
-	9250 1950 10100 1950
 $Comp
 L Jumper:Jumper_2_Open JP4
@@
 	8350 1250 8800 1250
 Wire Notes Line
-	11200 550  9950 550
-Wire Notes Line
-	9950 550  9950 2000
-Wire Notes Line
-	9950 2000 11200 2000
-Wire Notes Line
-	11200 550  11200 2000
-Wire Notes Line
 	9150 1300 9350 1300
 Wire Notes Line
 	9350 1300 9350 2000
-Wire Notes Line
-	9350 2000 9150 2000
 Wire Notes Line
 	9150 2000 9150 1300
@@
 $EndComp
 $Comp
-L LED:WS2812B D4
+L LED:WS2812B D2
 U 1 1 632689F9
 P 12600 6250
-F 0 "D4" H 12944 6296 50  0000 L CNN
+F 0 "D2" H 12944 6296 50  0000 L CNN
 F 1 "WS2812B" H 12944 6205 50  0000 L CNN
 F 2 "LED_SMD:LED_WS2812B_PLCC4_5.0x5.0mm_P3.2mm" H 12650 5950 50  0001 L TNN
@@
 $EndComp
 $Comp
-L LED:WS2812B D7
+L LED:WS2812B D3
 U 1 1 63277DB5
 P 13650 6250
-F 0 "D7" H 13994 6296 50  0000 L CNN
+F 0 "D3" H 13994 6296 50  0000 L CNN
 F 1 "WS2812B" H 13994 6205 50  0000 L CNN
 F 2 "LED_SMD:LED_WS2812B_PLCC4_5.0x5.0mm_P3.2mm" H 13700 5950 50  0001 L TNN
@@
 $EndComp
 $Comp
-L LED:WS2812B D10
+L LED:WS2812B D4
 U 1 1 63277F91
 P 14700 6250
-F 0 "D10" H 15044 6296 50  0000 L CNN
+F 0 "D4" H 15044 6296 50  0000 L CNN
 F 1 "WS2812B" H 15044 6205 50  0000 L CNN
 F 2 "LED_SMD:LED_WS2812B_PLCC4_5.0x5.0mm_P3.2mm" H 14750 5950 50  0001 L TNN
@@
 $EndComp
 $Comp
-L LED:WS2812B D2
+L LED:WS2812B D5
 U 1 1 63288C0E
 P 11550 7600
-F 0 "D2" H 11894 7646 50  0000 L CNN
+F 0 "D5" H 11894 7646 50  0000 L CNN
 F 1 "WS2812B" H 11894 7555 50  0000 L CNN
 F 2 "LED_SMD:LED_WS2812B_PLCC4_5.0x5.0mm_P3.2mm" H 11600 7300 50  0001 L TNN
@@
 $EndComp
 $Comp
-L LED:WS2812B D5
+L LED:WS2812B D6
 U 1 1 63288E2E
 P 12600 7600
-F 0 "D5" H 12944 7646 50  0000 L CNN
+F 0 "D6" H 12944 7646 50  0000 L CNN
 F 1 "WS2812B" H 12944 7555 50  0000 L CNN
 F 2 "LED_SMD:LED_WS2812B_PLCC4_5.0x5.0mm_P3.2mm" H 12650 7300 50  0001 L TNN
@@
 $EndComp
 $Comp
-L LED:WS2812B D8
+L LED:WS2812B D7
 U 1 1 63288E38
 P 13650 7600
-F 0 "D8" H 13994 7646 50  0000 L CNN
+F 0 "D7" H 13994 7646 50  0000 L CNN
 F 1 "WS2812B" H 13994 7555 50  0000 L CNN
 F 2 "LED_SMD:LED_WS2812B_PLCC4_5.0x5.0mm_P3.2mm" H 13700 7300 50  0001 L TNN
@@
 $EndComp
 $Comp
-L LED:WS2812B D11
+L LED:WS2812B D8
 U 1 1 63288E42
 P 14700 7600
-F 0 "D11" H 15044 7646 50  0000 L CNN
+F 0 "D8" H 15044 7646 50  0000 L CNN
 F 1 "WS2812B" H 15044 7555 50  0000 L CNN
 F 2 "LED_SMD:LED_WS2812B_PLCC4_5.0x5.0mm_P3.2mm" H 14750 7300 50  0001 L TNN
@@
 $EndComp
 $Comp
-L LED:WS2812B D3
+L LED:WS2812B D9
 U 1 1 6329CDBD
 P 11550 8950
-F 0 "D3" H 11894 8996 50  0000 L CNN
+F 0 "D9" H 11894 8996 50  0000 L CNN
 F 1 "WS2812B" H 11894 8905 50  0000 L CNN
 F 2 "LED_SMD:LED_WS2812B_PLCC4_5.0x5.0mm_P3.2mm" H 11600 8650 50  0001 L TNN
@@
 $EndComp
 $Comp
-L LED:WS2812B D6
+L LED:WS2812B D10
 U 1 1 6329D065
 P 12600 8950
-F 0 "D6" H 12944 8996 50  0000 L CNN
+F 0 "D10" H 12944 8996 50  0000 L CNN
 F 1 "WS2812B" H 12944 8905 50  0000 L CNN
 F 2 "LED_SMD:LED_WS2812B_PLCC4_5.0x5.0mm_P3.2mm" H 12650 8650 50  0001 L TNN
@@
 $EndComp
 $Comp
-L LED:WS2812B D9
+L LED:WS2812B D11
 U 1 1 6329D06F
 P 13650 8950
-F 0 "D9" H 13994 8996 50  0000 L CNN
+F 0 "D11" H 13994 8996 50  0000 L CNN
 F 1 "WS2812B" H 13994 8905 50  0000 L CNN
 F 2 "LED_SMD:LED_WS2812B_PLCC4_5.0x5.0mm_P3.2mm" H 13700 8650 50  0001 L TNN
@@
 Wire Wire Line
 	9050 7500 9300 7500
+$Comp
+L Switch:SW_SPDT SW1
+U 1 1 60E5AE6E
+P 10350 1350
+AR Path="/60E5AE6E" Ref="SW1"  Part="1"
+AR Path="/60E4053B/60E5AE6E" Ref="SW1"  Part="1"
+F 0 "SW1" H 10350 1025 50  0000 C CNN
+F 1 "SW_SPDT" H 10350 1116 50  0000 C CNN
+F 2 "Button_Switch_THT:SW_E-Switch_EG1224_SPDT_Angled" H 10350 1350 50  0001 C CNN
+F 3 "" H 10350 1350 50  0001 C CNN
+	1    10350 1350
+	-1   0    0    1
+$EndComp
+Wire Wire Line
+	9250 1950 10850 1950
+Wire Wire Line
+	10850 1650 10850 1950
+Wire Wire Line
+	10000 1250 10150 1250
+Connection ~ 10000 1250
+Wire Notes Line
+	9150 2000 9350 2000
 $EndSCHEMATC

Commit message: ordering
Parts:
- removed U1: MT8888CN1, buggyboy:SSOP-24_5.3x8.2mm_P0.65mm-HandSolder, symbol brains-rescue:MT8888C-buggyboy
- added C33, C34: 32pF, Capacitor_SMD:C_0402_1005Metric_Pad0.74x0.62mm_HandSolder, symbol Device:C_Small
- added C35: 100nF, Capacitor_SMD:C_0603_1608Metric_Pad1.08x0.95mm_HandSolder, symbol Device:C_Small
- added JP1: JUMP_XTAL_ALT, Jumper:SolderJumper-2_P1.3mm_Open_RoundedPad1.0x1.5mm, symbol Device:Jumper_NO_Small
- added R10: 2.2m, Resistor_SMD:R_0805_2012Metric_Pad1.20x1.40mm_HandSolder, symbol Device:R
- added U1: MT8888CS1, Package_SO:SOIC-20W_7.5x12.8mm_P1.27mm, symbol brains-rescue:MT8888CS1
- added U4: SN74LVC1GX04, Package_TO_SOT_SMD:SOT-563, symbol brains-rescue:SN74LVC1GX04
- added Y1: Crystal_Small, Crystal:Crystal_HC49-U_Vertical, symbol Device:Crystal_Small
- C10: footprint Capacitor_SMD:C_0805_2012Metric -> Capacitor_SMD:C_0603_1608Metric_Pad1.08x0.95mm_HandSolder
- C7: footprint Capacitor_SMD:C_0805_2012Metric -> Capacitor_SMD:C_0805_2012Metric_Pad1.18x1.45mm_HandSolder
Connections:
- net +5V: now also C35.1, U1.20 (VDD), U4.5 (VCC)
- net D0: now also U1.14 (D0)
- net D1: now also U1.15 (D1)
- net D2: now also U1.16 (D2)
- net D3: now also U1.17 (D3)
- net DTMF_IN: now also U1.2 (IN-)
- net GND: now also C33.1, C34.1, C35.2, U1.5 (VSS), U4.2 (GND)
- net TELCO_CS: now also U1.10 (CS)
- net TELCO_IRQ: now also U1.13 (!IRQ/CP)
- net TELCO_RD: now also U1.12 (RD)
- net TELCO_RS0: now also U1.11 (RS0)
- net TELCO_WR: now also U1.9 (WR)
- net at C2.2, C9.2, R5.2: now also U1.8 (TONE)
- net at R6.1: now also U1.18 (ESt)
- net at C4.2, R6.2: now also U1.19 (St/GT)
- net at R4.1: now also U1.3 (GS)
- net at TP3.1, X1.8 (OUT): now also JP1.2, U1.6 (OSC1)
- new net: U1.1 (IN+), U1.4 (VREF)
- new net: C33.2, R10.2, U4.3 (X1), Y1.1
- new net: C34.2, R10.1, U4.4 (X2), Y1.2
- new net XTAL_ALT: JP1.1, U4.6 (Y)
Changed lines of the file:
@@
-	1    0    0    -1
-$EndComp
-$Comp
-L brains-rescue:MT8888C-buggyboy U1
-U 1 1 60E5ACC4
-P 6200 1700
-AR Path="/60E5ACC4" Ref="U1"  Part="1"
-AR Path="/60E4053B/60E5ACC4" Ref="U1"  Part="1"
-F 0 "U1" H 6175 2615 50  0000 C CNN
-F 1 "MT8888CN1" H 6175 2524 50  0000 C CNN
-F 2 "buggyboy:SSOP-24_5.3x8.2mm_P0.65mm-HandSolder" H 6200 1650 50  0001 C CNN
-F 3 "" H 6200 1650 50  0001 C CNN
-	1    6200 1700
 	1    0    0    -1
 $EndComp
@@
 F 0 "C10" H 8692 7896 50  0000 L CNN
 F 1 "47nF" H 8692 7805 50  0000 L CNN
-F 2 "Capacitor_SMD:C_0805_2012Metric" H 8600 7850 50  0001 C CNN
+F 2 "Capacitor_SMD:C_0603_1608Metric_Pad1.08x0.95mm_HandSolder" H 8600 7850 50  0001 C CNN
 F 3 "~" H 8600 7850 50  0001 C CNN
 	1    8600 7850
@@
 Wire Wire Line
 	8600 8350 8600 8450
-Wire Wire Line
-	4100 1600 4700 1600
 $Comp
 L Connector_Generic:Conn_01x04 J2
@@
 F 0 "C7" V 8250 7250 50  0000 L CNN
 F 1 "10uF" V 8050 7200 50  0000 L CNN
-F 2 "Capacitor_SMD:C_0805_2012Metric" H 8150 7300 50  0001 C CNN
+F 2 "Capacitor_SMD:C_0805_2012Metric_Pad1.18x1.45mm_HandSolder" H 8150 7300 50  0001 C CNN
 F 3 "~" H 8150 7300 50  0001 C CNN
 	1    8150 7300
@@
 Wire Notes Line
 	9150 2000 9350 2000
+$Comp
+L brains-rescue:SN74LVC1GX04 U4
+U 1 1 63CEFE72
+P 10000 3750
+F 0 "U4" H 10000 4165 50  0000 C CNN
+F 1 "SN74LVC1GX04" H 10000 4074 50  0000 C CNN
+F 2 "Package_TO_SOT_SMD:SOT-563" H 10000 3600 50  0001 C CNN
+F 3 "" H 10000 3600 50  0001 C CNN
+	1    10000 3750
+	1    0    0    -1
+$EndComp
+$Comp
+L Device:R R10
+U 1 1 63CF2B84
+P 10000 3200
+F 0 "R10" V 9793 3200 50  0000 C CNN
+F 1 "2.2m" V 9884 3200 50  0000 C CNN
+F 2 "Resistor_SMD:R_0805_2012Metric_Pad1.20x1.40mm_HandSolder" V 9930 3200 50  0001 C CNN
+F 3 "~" H 10000 3200 50  0001 C CNN
+	1    10000 3200
+	0    1    1    0
+$EndComp
+$Comp
+L Device:Crystal_Small Y1
+U 1 1 63D0AD38
+P 10000 2800
+F 0 "Y1" H 10000 3025 50  0000 C CNN
+F 1 "Crystal_Small" H 10000 2934 50  0000 C CNN
+F 2 "Crystal:Crystal_HC49-U_Vertical" H 10000 2800 50  0001 C CNN
+F 3 "~" H 10000 2800 50  0001 C CNN
+	1    10000 2800
+	1    0    0    -1
+$EndComp
+$Comp
+L Device:C_Small C33
+U 1 1 63D0BBEF
+P 9700 2400
+F 0 "C33" H 9792 2446 50  0000 L CNN
+F 1 "32pF" H 9792 2355 50  0000 L CNN
+F 2 "Capacitor_SMD:C_0402_1005Metric_Pad0.74x0.62mm_HandSolder" H 9700 2400 50  0001 C CNN
+F 3 "~" H 9700 2400 50  0001 C CNN
+	1    9700 2400
+	1    0    0    -1
+$EndComp
+$Comp
+L Device:C_Small C34
+U 1 1 63D0C933
+P 10300 2400
+F 0 "C34" H 10392 2446 50  0000 L CNN
+F 1 "32pF" H 10392 2355 50  0000 L CNN
+F 2 "Capacitor_SMD:C_0402_1005Metric_Pad0.74x0.62mm_HandSolder" H 10300 2400 50  0001 C CNN
+F 3 "~" H 10300 2400 50  0001 C CNN
+	1    10300 2400
+	1    0    0    -1
+$EndComp
+Wire Wire Line
+	9700 2500 9700 2800
+Wire Wire Line
+	9700 2800 9900 2800
+Wire Wire Line
+	10300 2500 10300 2800
+Wire Wire Line
+	10300 2800 10100 2800
+Wire Wire Line
+	9700 2800 9700 3200
+Wire Wire Line
+	9700 3200 9850 3200
+Connection ~ 9700 2800
+Wire Wire Line
+	10300 2800 10300 3200
+Wire Wire Line
+	10300 3200 10150 3200
+Connection ~ 10300 2800
+Wire Wire Line
+	9700 3200 9550 3200
+Wire Wire Line
+	9550 3200 9550 3600
+Wire Wire Line
+	9550 3600 9650 3600
+Connection ~ 9700 3200
+Wire Wire Line
+	10300 3200 10450 3200
+Wire Wire Line
+	10450 3200 10450 3600
+Wire Wire Line
+	10450 3600 10350 3600
+Connection ~ 10300 3200
+$Comp
+L power:GND #PWR0136
+U 1 1 63DD5C34
+P 10700 2300
+AR Path="/63DD5C34" Ref="#PWR0136"  Part="1"
+AR Path="/60E4053B/63DD5C34" Ref="#PWR?"  Part="1"
+F 0 "#PWR0136" H 10700 2050 50  0001 C CNN
+F 1 "GND" V 10705 2172 50  0000 R CNN
+F 2 "" H 10700 2300 50  0001 C CNN
+F 3 "" H 10700 2300 50  0001 C CNN
+	1    10700 2300
+	1    0    0    -1
+$EndComp
+Wire Wire Line
+	9700 2300 10300 2300
+Connection ~ 10300 2300
+Wire Wire Line
+	10300 2300 10700 2300
+$Comp
+L power:GND #PWR0137
+U 1 1 63DEF237
+P 9500 3850
+AR Path="/63DEF237" Ref="#PWR0137"  Part="1"
+AR Path="/60E4053B/63DEF237" Ref="#PWR?"  Part="1"
+F 0 "#PWR0137" H 9500 3600 50  0001 C CNN
+F 1 "GND" V 9505 3722 50  0000 R CNN
+F 2 "" H 9500 3850 50  0001 C CNN
+F 3 "" H 9500 3850 50  0001 C CNN
+	1    9500 3850
+	1    0    0    -1
+$EndComp
+Wire Wire Line
+	9650 3750 9500 3750
+Wire Wire Line
+	9500 3750 9500 3850
+$Comp
+L power:+5V #PWR0138
+U 1 1 63E2144A
+P 10850 3750
+AR Path="/63E2144A" Ref="#PWR0138"  Part="1"
+AR Path="/60E4053B/63E2144A" Ref="#PWR?"  Part="1"
+F 0 "#PWR0138" H 10850 3600 50  0001 C CNN
+F 1 "+5V" V 10865 3878 50  0000 L CNN
+F 2 "" H 10850 3750 50  0001 C CNN
+F 3 "" H 10850 3750 50  0001 C CNN
+	1    10850 3750
+	0    1    1    0
+$EndComp
+$Comp
+L Device:C_Small C35
+U 1 1 63E3CC40
+P 10800 3900
+F 0 "C35" H 10892 3946 50  0000 L CNN
+F 1 "100nF" H 10892 3855 50  0000 L CNN
+F 2 "Capacitor_SMD:C_0603_1608Metric_Pad1.08x0.95mm_HandSolder" H 10800 3900 50  0001 C CNN
+F 3 "~" H 10800 3900 50  0001 C CNN
+	1    10800 3900
+	1    0    0    -1
+$EndComp
+Wire Wire Line
+	10350 3750 10800 3750
+Wire Wire Line
+	10800 3750 10800 3800
+Connection ~ 10800 3750
+Wire Wire Line
+	10800 3750 10850 3750
+$Comp
+L power:GND #PWR0139
+U 1 1 63E6C67D
+P 10800 4050
+AR Path="/63E6C67D" Ref="#PWR0139"  Part="1"
+AR Path="/60E4053B/63E6C67D" Ref="#PWR?"  Part="1"
+F 0 "#PWR0139" H 10800 3800 50  0001 C CNN
+F 1 "GND" V 10805 3922 50  0000 R CNN
+F 2 "" H 10800 4050 50  0001 C CNN
+F 3 "" H 10800 4050 50  0001 C CNN
+	1    10800 4050
+	1    0    0    -1
+$EndComp
+Wire Wire Line
+	10800 4000 10800 4050
+Wire Wire Line
+	10350 3900 10650 3900
+Text Label 10650 3900 2    50   ~ 0
+XTAL_ALT
+$Comp
+L Device:Jumper_NO_Small JP1
+U 1 1 63EA4290
+P 4350 1250
+F 0 "JP1" V 4304 1298 50  0000 L CNN
+F 1 "JUMP_XTAL_ALT" V 4395 1298 50  0000 L CNN
+F 2 "Jumper:SolderJumper-2_P1.3mm_Open_RoundedPad1.0x1.5mm" H 4350 1250 50  0001 C CNN
+F 3 "~" H 4350 1250 50  0001 C CNN
+	1    4350 1250
+	0    1    1    0
+$EndComp
+Wire Wire Line
+	4100 1600 4350 1600
+Wire Wire Line
+	4350 1350 4350 1600
+Connection ~ 4350 1600
+Wire Wire Line
+	4350 1600 4700 1600
+Wire Wire Line
+	4350 1150 4350 850
+Text Label 4350 850  2    50   ~ 0
+XTAL_ALT
+$Comp
+L brains-rescue:MT8888CS1 U1
+U 1 1 629A2883
+P 6200 1700
+F 0 "U1" H 6175 2615 50  0000 C CNN
+F 1 "MT8888CS1" H 6175 2524 50  0000 C CNN
+F 2 "Package_SO:SOIC-20W_7.5x12.8mm_P1.27mm" H 6200 1650 50  0001 C CNN
+F 3 "" H 6200 1650 50  0001 C CNN
+	1    6200 1700
+	1    0    0    -1
+$EndComp
 $EndSCHEMATC
