File: hardware/buggyboy/keypad.kicad_pcb (KiCad board)
At the start: 2 copper layers, 88 x 132 mm, 48 parts, among them J1 Conn_01x12, U1 HD44780, U2 74LS166, U3 74LS166

Commit message: ordering
Parts:
- added H3: MNT3, MountingHole:MountingHole_4.3mm_M4_Pad_Via, F.Cu at (187.0, 35.0)
- added H4: MNT4, MountingHole:MountingHole_4.3mm_M4_Pad_Via, F.Cu at (109.0, 35.0)
- R1, R10, R11, R12, R13, R14, R15, R16, R17, R18, R19, R2, R20, R21, R22, R23, R3, R4, R5, R6, R7, R8, R9: footprint Resistor_THT:R_Axial_DIN0204_L3.6mm_D1.6mm_P7.62mm_Horizontal -> Resistor_SMD:R_0603_1608Metric_Pad0.98x0.95mm_HandSolder
- SW_0, SW_1, SW_2, SW_3, SW_4, SW_5, SW_6, SW_7, SW_8, SW_9, SW_A1, SW_B1, SW_C1, SW_D1, SW_OCTO1, SW_STAR1: footprint Button_Switch_Keyboard:SW_Cherry_MX1A_1.00u_PCB -> Button_Switch_Keyboard:SW_Cherry_MX_1.00u_PCB
- U1: footprint Display:WC1602A -> buggyboy:WC1602A
- moved R21 2.51 mm to (182.0, 48.8)
- moved R18 0.50 mm to (111.5, 48.0), turned to 45 degrees
Connections:
- U1 pad 10: (no net) -> Net-(U1-Pad10)
- U1 pad 7: (no net) -> Net-(U1-Pad7)
- U1 pad 8: (no net) -> Net-(U1-Pad8)
- U1 pad 9: (no net) -> Net-(U1-Pad9)
Routing:
- net +5V: track 716.2 -> 728.2 mm, vias 0 -> 2
- net Net-(R23-Pad2): track 4.07 -> 8.44 mm
- net Net-(R7-Pad1): track 52.8 -> 55.7 mm
- net Net-(R21-Pad1): track 4.12 -> 6.17 mm, vias 0 -> 1
- net Net-(R18-Pad1): track 4.97 -> 6.99 mm, vias 0 -> 1
- net Net-(R14-Pad1): track 99.8 -> 101.5 mm
- net Net-(R16-Pad1): track 86.1 -> 87.8 mm
- net Net-(R6-Pad1): track 66.6 -> 65.0 mm
- net Net-(R1-Pad1): track 34.9 -> 35.8 mm
- net Net-(R5-Pad1): track 43.0 -> 43.8 mm
- net Net-(R13-Pad1): track 57.0 -> 56.4 mm
- net Net-(R19-Pad1): track 5.12 -> 5.59 mm, vias 0 -> 1
- net Net-(R22-Pad1): track 5.38 -> 5.83 mm, vias 0 -> 1
- net GND: vias 21 -> 29
Other:
- board text added: "USE M3 SCREWS"
- board text added: "V2.1"
- board text removed: "V2.0"
