File: hardware/buggyboy/keypad.sch (KiCad schematic (older format))
At the start: 48 parts, among them J1 Conn_01x12, U1 HD44780, U2 74LS166, U3 74LS166

Commit message: ordering
Parts:
- U1: footprint Display:WC1602A -> buggyboy:WC1602A
Changed lines of the file:
@@
 F 0 "U1" H 5050 2665 50  0000 C CNN
 F 1 "HD44780" H 5050 2574 50  0000 C CNN
-F 2 "Display:WC1602A" H 5050 1800 50  0001 C CNN
+F 2 "buggyboy:WC1602A" H 5050 1800 50  0001 C CNN
 F 3 "" H 5050 1800 50  0001 C CNN
 	1    5050 1800
